File: pi-crust.brd (EAGLE design)
At the start: 43.7 x 40.4 mm, 11 parts

Commit message: Special edition PS1 silkscreen
Parts:
- added U$2: LOGO, E-test-solutions (6):LOGO
Other:
- board text removed: "Pi Crust v5"
Changed lines of the file:
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@@
 <rectangle x1="42.418" y1="20.828" x2="43.942" y2="22.352" layer="26"/>
 <rectangle x1="28.194" y1="6.604" x2="29.718" y2="8.128" layer="26"/>
-<text x="15.771271875" y="11.068684375" size="2.032" layer="25" font="vector" ratio="12" rot="R90">Pi Crust v5</text>
-<text x="18.17261875" y="11.083584375" size="1.651" layer="25" font="vector" rot="R90">picru.st/</text>
+<text x="15.14951875" y="1.22743125" size="1.651" layer="25" font="vector" rot="R90">picru.st/</text>
 <text x="14.08355" y="1.54111875" size="1.27" layer="26" font="vector" rot="MR90">by @joewalnes (CC-SA) </text>
 <wire x1="10.16" y1="40.386" x2="10.16" y2="33.528" width="0.127" layer="27"/>
@@
 <attribute name="VALUE" x="3.81" y="34.925" size="1.27" layer="27"/>
 </element>
+<element name="U$2" library="E-test-solutions (6)" package="LOGO" value="LOGO" x="17.2212" y="21.59"/>
 </elements>
 <signals>
@@
 </signal>
 </signals>
-<errors>
-</errors>
 </board>
 </drawing>
